File: testdrive/hw/Pendu.kicad_pcb (KiCad board)
At the start: 2 copper layers, 36 x 20 mm, 26 parts, among them J1 Conn_01x04, J2 Conn_01x08, J3 Conn_01x05, J4 Conn_01x05, Q1 Si2301DS, SW1 Vib, U1 SPX3819M5-L-3-3, U2 STM32G030F6Px, U3 BMI270, U4 MMC5603NJ

Commit message: Fix circuit design, submit for fabrication
Parts:
- added G***: LOGO, LOGO, B.Cu at (24.1, 45.5)
- added G***: LOGO, LOGO, B.Cu at (36.8, 47.0)
- added Q2: Si2301DS, Package_TO_SOT_SMD:SOT-23, F.Cu at (38.6, 32.3)
- added R2: 1.2M, Resistor_SMD:R_0603_1608Metric, F.Cu at (41.2, 32.7)
- moved C1 1.13 mm to (40.1, 36.9)
- moved SW1 0.77 mm to (43.9, 32.8)
- moved U1 0.77 mm to (48.2, 32.8)
- moved R1 0.52 mm to (39.4, 39.4)
- moved Q1 0.20 mm to (37.5, 36.2)
- renumbered R2 to R3, R3 to R4, R4 to R5, R5 to R6, R6 to R7
Connections:
- net VA|BAT renamed VBAT
- Q1 pad 1: PWR_LATCH -> Net-(Q1-G)
- R1 pad 1: PWR_LATCH -> Net-(Q1-G)
- SW1 pad 1: PWR_LATCH -> Net-(Q1-G)
- U2 pad 12: unconnected-(U2-PA5-Pad12) -> PWR_LATCH
Routing:
- net Net-(Q1-G): track 0.00 -> 11.9 mm
- net VDD: track 96.9 -> 89.3 mm, vias 6 -> 4
- net VBAT: track 11.0 -> 15.1 mm, vias 0 -> 2
- net PWR_LATCH: track 11.9 -> 15.4 mm
- net Net-(U1-BP): track 8.84 -> 9.84 mm
- net Net-(Q1-D): track 17.3 -> 17.9 mm
- net GND: vias 7 -> 6
Other:
- board text added: "23-WnSolst"
- board text added: "JLCJLCJLCJLC"
- board text added: "La pensée"
- board text added: "Rev. 1"
