File: mallet/hw/Mallet.kicad_pcb (KiCad board)
At the start: 2 copper layers, 0 parts

Commit message: Finish mallet PCB
Parts:
- added C1: 4.7u, Capacitor_SMD:C_0603_1608Metric, B.Cu at (22.5, 21.4)
- added C2: 100n, Capacitor_SMD:C_0603_1608Metric, B.Cu at (24.0, 21.4)
- added C3: 100n, Capacitor_SMD:C_0603_1608Metric, B.Cu at (27.1, 29.2)
- added C4: 10n, Capacitor_SMD:C_0603_1608Metric, F.Cu at (22.9, 30.7)
- added C5: 470n, Capacitor_SMD:C_0603_1608Metric, F.Cu at (31.1, 39.1)
- added C6: 100n, Capacitor_SMD:C_0603_1608Metric, F.Cu at (20.4, 33.1)
- added C7: 10u, Capacitor_SMD:CP_Elec_5x3.9, F.Cu at (25.9, 23.7)
- added D1: White, LED_SMD:LED_0603_1608Metric, F.Cu at (36.1, 40.6)
- added G***: LOGO, LOGO, B.Cu at (30.6, 39.1)
- added G***: LOGO, LOGO, B.Cu at (35.0, 38.9)
- added G***: LOGO, LOGO, B.Cu at (19.9, 30.4)
- added H1: MountingHole, Mallet_footprints:MountingHoles_M3_Tri14.5, F.Cu at (31.5, 28.2)
- added J1: Conn_01x05, Connector_PinHeader_2.00mm:PinHeader_1x05_P2.00mm_Vertical, F.Cu at (19.6, 24.4)
- added J2: Conn_01x05, Connector_PinHeader_2.00mm:PinHeader_1x05_P2.00mm_Vertical, F.Cu at (20.8, 24.4)
- added J3: Conn_01x03, Connector_PinHeader_2.00mm:PinHeader_1x03_P2.00mm_Vertical, F.Cu at (20.0, 39.6)
- added J4: Conn_01x04, Connector_PinHeader_2.00mm:PinHeader_1x04_P2.00mm_Vertical, F.Cu at (36.6, 25.2)
- added J5: Conn_01x04, Mallet_footprints:TestPoints_1x04_P2.0, F.Cu at (28.3, 16.2)
- added JP1: SolderJumper_2_Open, Jumper:SolderJumper-2_P1.3mm_Open_RoundedPad1.0x1.5mm, F.Cu at (33.2, 38.9)
- added R1: 1M, Resistor_SMD:R_0603_1608Metric, B.Cu at (34.6, 16.2)
- added R2: 1.5k, Resistor_SMD:R_0603_1608Metric, B.Cu at (32.3, 32.5)
- added R3: 1.5k, Resistor_SMD:R_0603_1608Metric, B.Cu at (33.8, 32.5)
- added R4: 6.8k, Resistor_SMD:R_0603_1608Metric, F.Cu at (36.1, 39.1)
- added R5: 220, Resistor_SMD:R_0603_1608Metric, F.Cu at (34.1, 26.4)
- added R6: 220, Resistor_SMD:R_0603_1608Metric, F.Cu at (34.1, 28.1)
- added R7: 220, Resistor_SMD:R_0603_1608Metric, F.Cu at (34.1, 29.9)
- added U1: STM32G030F6Px, Package_SO:TSSOP-20_4.4x6.5mm_P0.65mm, B.Cu at (28.6, 20.7)
- added U2: AS5600L-ASOM, Mallet_footprints:SOIC127P600X175-8N, B.Cu at (31.5, 28.2)
- added U3: DRV8313PWPR, Mallet_footprints:SOP65P640X120-29N, F.Cu at (25.9, 36.4)
Routing:
- net +3.3V: track 0.00 -> 44.4 mm, vias 0 -> 1
- net LED_ACT: track 0.00 -> 39.7 mm, vias 0 -> 1
- net EN: track 0.00 -> 27.5 mm, vias 0 -> 1
- net NSLEEP: track 0.00 -> 27.2 mm, vias 0 -> 1
- net NFAULT: track 0.00 -> 25.6 mm, vias 0 -> 1
- net IN_U: track 0.00 -> 20.4 mm, vias 0 -> 1
- net IN_V: track 0.00 -> 17.7 mm, vias 0 -> 1
- net MAG_SDA: track 0.00 -> 14.8 mm
- net IN_W: track 0.00 -> 14.8 mm, vias 0 -> 1
- net MAG_SCL: track 0.00 -> 14.6 mm
- net UNIT_SDA: track 0.00 -> 14.3 mm, vias 0 -> 1
- net LED_B: track 0.00 -> 13.6 mm, vias 0 -> 1
- net SWCLK: track 0.00 -> 13.1 mm
- net UNIT_SCL: track 0.00 -> 11.6 mm
- net LED_R: track 0.00 -> 10.4 mm, vias 0 -> 1
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- added copper zone on B.Cu, net +3.3V
- added copper zone on B.Cu, net GND
- added copper zone on F.Cu, net GND
- added copper zone on F.Cu, net V3P3O
- added copper zone on F.Cu, net VM
Other:
- board outline added: 19.5 x 27 mm
- board text added: "G"
- board text added: "JLCJLCJLCJLC"
- board text added: "L"
- board text added: "M"
- board text added: "Mallet Rev. 1"
- board text added: "Malletwand"
- board text added: "SCL"
- board text added: "SDA"
- board text added: "U"
- board text added: "V"
- board text added: "W"
