File: wand/hw/Wand.kicad_sch (KiCad schematic)
At the start: 65 parts, among them J2 Conn_01x03, J2 Conn_01x04, J3 Conn_01x03, J4 Conn_01x04, J5 Conn_01x04, J6 USB_C_Receptacle_PowerOnly_6P, M1 Vib, Q1 Si2301, Q2 Si2302, SW1 SW_SPST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

Commit message: 🚧 Updating circuit board design
Parts:
- R4, R5, R6: footprint Resistor_SMD:R_0603_1608Metric -> Resistor_SMD:R_0402_1005Metric
Connections:
- net LED_B: now also U3.5 (PA0); no longer U3.15 (PA10)
- net LED_R: now also U3.15 (PA10); no longer U3.5 (PA0)
- net BMI_MISO: no longer names the net of U3.9 (PA6)
- net BMI_MISO: no longer U4.1 (SDO)
- no-connect marks 19 -> 21
Changed lines of the file:
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@@
   (no_connect (at 66.04 90.17))
   (no_connect (at 230.505 82.55))
+  (no_connect (at 230.505 74.93))
   (no_connect (at 260.985 74.93))
   (no_connect (at 66.04 87.63))
   (no_connect (at 307.975 60.325))
+  (no_connect (at 330.835 52.705))
   (no_connect (at 307.975 57.785))
   (no_connect (at 307.975 50.165))
@@
     (stroke (width 0) (type default))
   )
-  (wire (pts (xy 230.505 72.39) (xy 230.505 74.93))
-    (stroke (width 0) (type default))
-  )
   (wire (pts (xy -23.495 27.305) (xy -24.765 27.305))
     (stroke (width 0) (type default))
@@
     )
   )
-  (global_label "LED_B" (shape bidirectional) (at 330.835 60.325 0) (fields_autoplaced)
+  (global_label "LED_R" (shape bidirectional) (at 330.835 60.325 0) (fields_autoplaced)
     (effects (font (size 1.27 1.27)) (justify left))
     (property "Intersheetrefs" "${INTERSHEET_REFS}" (at 340.6162 60.325 0)
@@
     )
   )
-  (global_label "BMI_MISO" (shape bidirectional) (at 330.835 52.705 0) (fields_autoplaced)
-    (effects (font (size 1.27 1.27)) (justify left))
-    (property "Intersheetrefs" "${INTERSHEET_REFS}" (at 343.8215 52.705 0)
-      (effects (font (size 1.27 1.27)) (justify left) hide)
-    )
-  )
   (global_label "LED_G" (shape bidirectional) (at 330.835 45.085 0) (fields_autoplaced)
     (effects (font (size 1.27 1.27)) (justify left))
@@
     )
   )
-  (global_label "LED_R" (shape bidirectional) (at 330.835 42.545 0) (fields_autoplaced)
+  (global_label "LED_B" (shape bidirectional) (at 330.835 42.545 0) (fields_autoplaced)
     (effects (font (size 1.27 1.27)) (justify left))
     (property "Intersheetrefs" "${INTERSHEET_REFS}" (at 340.6162 42.545 0)
@@
     )
   )
-  (global_label "BMI_MISO" (shape bidirectional) (at 230.505 72.39 180) (fields_autoplaced)
-    (effects (font (size 1.27 1.27)) (justify right))
-    (property "Intersheetrefs" "${INTERSHEET_REFS}" (at 217.5185 72.39 0)
-      (effects (font (size 1.27 1.27)) (justify right) hide)
-    )
-  )
   (global_label "BMI_SCK" (shape bidirectional) (at 245.745 62.865 90) (fields_autoplaced)
     (effects (font (size 1.27 1.27)) (justify left))
@@
       (effects (font (size 1.27 1.27)))
     )
-    (property "Footprint" "Resistor_SMD:R_0603_1608Metric" (at 233.68 35.052 90)
+    (property "Footprint" "Resistor_SMD:R_0402_1005Metric" (at 233.68 35.052 90)
       (effects (font (size 1.27 1.27)) hide)
     )
@@
       (effects (font (size 1.27 1.27)))
     )
-    (property "Footprint" "Resistor_SMD:R_0603_1608Metric" (at 233.68 37.592 90)
+    (property "Footprint" "Resistor_SMD:R_0402_1005Metric" (at 233.68 37.592 90)
       (effects (font (size 1.27 1.27)) hide)
     )
@@
       (effects (font (size 1.27 1.27)))
     )
-    (property "Footprint" "Resistor_SMD:R_0603_1608Metric" (at 233.68 29.972 90)
-      (effects (font (size 1.27 1.27)) hide)
-    )
+    (property "Footprint" "Resistor_SMD:R_0402_1005Metric" (at 233.68 29.972 90)
+      (effects (font (size 1.27 1.27)) hide)
+    )
