File: wand/hw/Wand.kicad_pcb (KiCad board)
At the start: 2 copper layers, 63.2 x 22.8 mm, 64 parts, among them J1 Conn_01x04, J2 Conn_01x08, J3 Conn_01x08, J4 Conn_01x04, J5 USB_C_Receptacle_PowerOnly_6P, M1 Vib, Q1 Si2301, Q2 Si2302, SW1 SW_SPST, SW2 Vib, U1 SPX3819M5-L-3-3, U2 STM32G030F6Px, U3 BMI270, U4 MMC5603NJ, U5 nRF24L01P, U6 LTC4054ES5-4.2, Y1 16MHz

Commit message: 🚧 Updating circuit board design
Parts:
- added C5: 10u, Capacitor_SMD:C_0402_1005Metric, B.Cu at (48.9, 47.8)
- added C6: 100n, Capacitor_SMD:C_0402_1005Metric, B.Cu at (48.9, 46.9)
- added C7: 100n, Capacitor_SMD:C_0402_1005Metric, B.Cu at (48.5, 42.4)
- added J4: Conn_01x04, Wand_footprints:TestPoints_1x04_P2.0, F.Cu at (44.7, 44.6)
- added U3: STM32L011F4Ux, Package_DFN_QFN:ST_UFQFPN-20_3x3mm_P0.5mm, B.Cu at (48.8, 44.6)
- J2, J3: value Conn_01x08 -> Conn_01x03; footprint Connector_PinHeader_1.00mm:PinHeader_1x08_P1.00mm_Vertical -> Connector_PinHeader_1.00mm:PinHeader_1x03_P1.00mm_Vertical
- R4, R5, R6: value 1k TBD -> 2k TBD
- moved R3 20.2 mm to (35.7, 47.2), turned to 0 degrees
- moved R2 17.6 mm to (35.7, 44.7), turned to 0 degrees
- moved R4 9.80 mm to (48.2, 46.2), turned to 180 degrees
- moved R5 7.51 mm to (48.2, 44.1), turned to 180 degrees
- moved R6 6.08 mm to (48.2, 42.6), turned to 180 degrees
- moved C10 5.19 mm to (53.8, 47.6), turned to 90 degrees
- moved U5 4.73 mm to (51.9, 48.0), turned to 180 degrees
- moved C8 3.68 mm to (54.2, 43.4), turned to -90 degrees
- moved C9 3.33 mm to (54.2, 45.3), turned to 90 degrees
- moved J3 2.56 mm to (50.9, 41.3)
- moved J2 2.48 mm to (50.9, 39.0)
- moved J5 0.73 mm to (46.3, 46.2)
- moved U4 0.31 mm to (51.9, 44.5), turned to 90 degrees
- renumbered C7 to C10, C8 to C11, C9 to C12, C10 to C13, C11 to C14, C12 to C15, C13 to C16, C14 to C17, C15 to C18, C16 to C19, C17 to C20, C18 to C21, C19 to C22, C20 to C23, C5 to C8, C6 to C9, J4 to J5, J5 to J6, U3 to U4, U4 to U5, U5 to U6, U6 to U7
Connections:
- net SPI1_MISO renamed nRF_MISO
- net SWCLK renamed HSWCLK
- net SWDIO renamed HSWDIO
- C11 pad 1: VBAT -> VDD
- J2 pad 3: SPI2_MOSI -> BOB_DA
- J3 pad 3: SPI2_MOSI -> BOB_DA
- J5 pad 1: LED_R -> Net-(J5-Pin_1)
- J5 pad 3: LED_G -> Net-(J5-Pin_3)
- J5 pad 4: LED_B -> Net-(J5-Pin_4)
- R2 pad 1: Net-(U2-PA12/PA10) -> BOB_DA
- R2 pad 2: SPI2_MOSI -> VDDSUB
- R4 pad 1: LED_B -> Net-(J5-Pin_1)
- R4 pad 2: Net-(U2-PB0/PB1/PB2/PA8) -> LED_R
- R5 pad 1: LED_G -> Net-(J5-Pin_3)
- R5 pad 2: Net-(U2-PB3/PB4/PB5/PB6) -> LED_G
- R6 pad 1: LED_R -> Net-(J5-Pin_4)
- R6 pad 2: Net-(U2-PB7/PB8) -> LED_B
- R7 pad 2: VBAT -> VDD
- U2 pad 1: Net-(U2-PB7/PB8) -> unconnected-(U2-PB7/PB8-Pad1)
- U2 pad 10: BMI_CS -> SUB_VDD_G
- U2 pad 12: VIB_TRG -> nRF_SCK
- U2 pad 14: nRF_CS -> nRF_MOSI
- U2 pad 15: Net-(U2-PB0/PB1/PB2/PA8) -> unconnected-(U2-PB0/PB1/PB2/PA8-Pad15)
- U2 pad 16: nRF_CE -> nRF_CS
- U2 pad 17: Net-(U2-PA12/PA10) -> nRF_CE
- U2 pad 2: SUB_VDD_G -> unconnected-(U2-PC14/PB9-Pad2)
- U2 pad 20: Net-(U2-PB3/PB4/PB5/PB6) -> unconnected-(U2-PB3/PB4/PB5/PB6-Pad20)
- U2 pad 7: SPI2_SCK -> VIB_TRG
- U2 pad 8: SPI1_SCK -> unconnected-(U2-PA1-Pad8)
- U2 pad 9: SPI1_MOSI -> BOB_DA
- U4 pad 1: unconnected-(U3-SDO-Pad1) -> BMI_MISO
- U4 pad 13: SPI2_SCK -> BMI_SCK
- U4 pad 14: SPI2_MOSI -> BMI_MOSI
- U6 pad 3: SPI1_SCK -> nRF_SCK
- U6 pad 4: SPI1_MOSI -> nRF_MOSI
Routing:
- net VDDSUB: track 31.1 -> 9.24 mm, vias 1 -> 0
- net SPI2_SCK: track 16.3 -> 0.00 mm, vias 1 -> 0
- net BMI_CS: track 14.7 -> 0.00 mm, vias 1 -> 0
- net unconnected-(U2-PB3/PB4/PB5/PB6-Pad20): track 0.00 -> 14.5 mm, vias 0 -> 2
- net Net-(U2-PB3/PB4/PB5/PB6): track 14.5 -> 0.00 mm, vias 2 -> 0
- net Net-(U2-PB0/PB1/PB2/PA8): track 14.4 -> 0.00 mm, vias 2 -> 0
- net LED_R: track 12.2 -> 0.00 mm
- net Net-(U2-PB7/PB8): track 12.1 -> 0.00 mm, vias 2 -> 0
- net LED_G: track 11.4 -> 0.00 mm
- net VBAT: track 18.8 -> 7.62 mm
- net LED_B: track 11.0 -> 0.00 mm
- net SUB_VDD_G: track 10.4 -> 0.00 mm, vias 2 -> 0
- net Net-(U2-PA12/PA10): track 10.2 -> 0.00 mm
- net SPI1_MOSI: track 9.90 -> 0.00 mm, vias 2 -> 0
- net SPI1_SCK: track 9.79 -> 0.00 mm, vias 2 -> 0
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Other:
- board size 63.2 x 22.8 mm -> 63.2 x 23.8 mm

Commit message: 🚧 Updating circuit board design
Parts:
- R4, R5, R6: footprint Resistor_SMD:R_0603_1608Metric -> Resistor_SMD:R_0402_1005Metric
- moved R3 20.3 mm to (51.8, 34.7)
- moved R2 17.3 mm to (49.3, 33.9), turned to -90 degrees
- moved R5 0.67 mm to (47.7, 43.6), turned to 0 degrees
- moved R6 0.58 mm to (47.7, 42.3), turned to 0 degrees
- moved R4 0.46 mm to (47.8, 46.1), turned to 0 degrees
Connections:
- U3 pad 15: LED_B -> LED_R
- U3 pad 5: LED_R -> LED_B
- U3 pad 9: BMI_MISO -> unconnected-(U3-PA6-Pad9)
- U4 pad 1: BMI_MISO -> unconnected-(U4-SDO-Pad1)
Routing:
- net VDDSUB: track 9.24 -> 51.7 mm, vias 0 -> 2
- net BOB_DA: track 0.00 -> 18.3 mm, vias 0 -> 1
- net unconnected-(U2-PB3/PB4/PB5/PB6-Pad20): track 14.5 -> 0.00 mm, vias 2 -> 0
- net BSWCLK: track 0.00 -> 10.0 mm, vias 0 -> 1
- net nRF_SCK: track 0.00 -> 7.61 mm, vias 0 -> 2
- net GND: track 32.7 -> 38.8 mm, vias 154 -> 156
- net BSWDIO: track 0.00 -> 3.75 mm
- net LED_B: track 0.00 -> 3.29 mm, vias 0 -> 1
- net BMI_MOSI: track 0.00 -> 3.22 mm, vias 0 -> 1
- net VDD: track 71.0 -> 73.8 mm
- net LED_G: track 0.00 -> 2.76 mm, vias 0 -> 1
- net LED_R: track 0.00 -> 2.12 mm, vias 0 -> 1
- net BMI_SCK: track 0.00 -> 2.12 mm, vias 0 -> 1
- net BMI_CS: track 0.00 -> 1.61 mm, vias 0 -> 1
- net SUB_VDD_G: track 0.00 -> 1.45 mm
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
Commit message: Finish wand board update
Parts:
- removed the G*** at (25.4, 38.6)
- moved U5 0.22 mm to (51.8, 47.8)
- moved U4 0.20 mm to (51.9, 44.3)
- moved C8 0.20 mm to (54.2, 43.2)
- moved C9 0.20 mm to (54.2, 45.1)
- moved C10 0.10 mm to (53.7, 47.6)
- moved R6 0.06 mm to (47.8, 42.4)
Routing:
- net LED_B: track 3.29 -> 2.23 mm
Other:
- outline, holes or cut-outs redrawn
- board text added: "24-Soak"
- board text added: "Wand Rev. 4"
- board text removed: "Wand Rev. 3"
